File: lab2_meres2.sch (KiCad schematic (older format))
At the start: 10 parts, among them J1 Conn_01x05_Female

Commit message: TL082 SPICE fájlok
Parts:
- removed R2: 1k, symbol Device:R
- removed R4: 100k, symbol Device:R
- C1: Spice_Model (none) -> 470n; Spice_Netlist_Enabled (none) -> Y; Spice_Primitive (none) -> C
- J1: Spice_Model (none) -> Conn_01x05_Female; Spice_Netlist_Enabled (none) -> N; Spice_Primitive (none) -> J
- R1: Spice_Model (none) -> 4.7k; Spice_Netlist_Enabled (none) -> Y; Spice_Primitive (none) -> R
- R3: Spice_Model (none) -> 47k; Spice_Netlist_Enabled (none) -> Y; Spice_Primitive (none) -> R
- U?: Spice_Lib_File adtl082_for_the_win.lib -> TL082.lib; Spice_Model 0 -> TL082; Spice_Node_Sequence (none) -> 1 2 4 5 3; Spice_Primitive R -> X
- V2, V3: Spice_Model dc 15 -> dc 10
Connections:
- wire segments 47 -> 46
Changed lines of the file:
@@
 $EndDescr
-$Comp
-L Device:C C1
-U 1 1 60228247
-P 2150 1500
-F 0 "C1" V 1898 1500 50  0000 C CNN
-F 1 "470n" V 1989 1500 50  0000 C CNN
-F 2 "" H 2188 1350 50  0001 C CNN
-F 3 "~" H 2150 1500 50  0001 C CNN
-	1    2150 1500
-	0    1    1    0
-$EndComp
 $Comp
 L Device:R R1
@@
 F 2 "" V 2580 1500 50  0001 C CNN
 F 3 "~" H 2650 1500 50  0001 C CNN
+F 4 "R" H 2650 1500 50  0001 C CNN "Spice_Primitive"
+F 5 "4.7k" H 2650 1500 50  0001 C CNN "Spice_Model"
+F 6 "Y" H 2650 1500 50  0001 C CNN "Spice_Netlist_Enabled"
 	1    2650 1500
 	0    1    1    0
@@
 F 2 "" V 4180 1500 50  0001 C CNN
 F 3 "~" H 4250 1500 50  0001 C CNN
+F 4 "R" H 4250 1500 50  0001 C CNN "Spice_Primitive"
+F 5 "47k" H 4250 1500 50  0001 C CNN "Spice_Model"
+F 6 "Y" H 4250 1500 50  0001 C CNN "Spice_Netlist_Enabled"
 	1    4250 1500
 	0    1    1    0
 $EndComp
-$Comp
-L Device:R R2
-U 1 1 60229439
-P 3500 2650
-F 0 "R2" H 3430 2604 50  0000 R CNN
-F 1 "1k" H 3430 2695 50  0000 R CNN
-F 2 "" V 3430 2650 50  0001 C CNN
-F 3 "~" H 3500 2650 50  0001 C CNN
-	1    3500 2650
-	-1   0    0    1
-$EndComp
-$Comp
-L Device:R R4
-U 1 1 602298B6
-P 4800 2500
-F 0 "R4" H 4730 2454 50  0000 R CNN
-F 1 "100k" H 4730 2545 50  0000 R CNN
-F 2 "" V 4730 2500 50  0001 C CNN
-F 3 "~" H 4800 2500 50  0001 C CNN
-	1    4800 2500
-	-1   0    0    1
-$EndComp
 Wire Wire Line
 	2800 1500 3650 1500
-Wire Wire Line
-	3500 2500 3500 1950
 Wire Wire Line
 	3500 1950 3850 1950
@@
 Wire Wire Line
 	3650 1500 4100 1500
-Wire Wire Line
-	2300 1500 2500 1500
 Wire Wire Line
 	4800 2050 4800 1500
@@
 	1    0    0    -1
 $EndComp
-Wire Wire Line
-	3500 2800 3500 3000
 Connection ~ 3500 3000
 Wire Wire Line
@@
 F 2 "" H 6100 950 50  0001 C CNN
 F 3 "~" H 6100 950 50  0001 C CNN
+F 4 "J" H 6100 950 50  0001 C CNN "Spice_Primitive"
+F 5 "Conn_01x05_Female" H 6100 950 50  0001 C CNN "Spice_Model"
+F 6 "N" H 6100 950 50  0001 C CNN "Spice_Netlist_Enabled"
 	1    6100 950
 	1    0    0    -1
@@
 	1600 1500 1600 1150
 Connection ~ 1600 1500
-Wire Wire Line
-	1600 1500 2000 1500
 Wire Wire Line
 	4050 750  4050 1750
@@
 F 3 "~" H 6400 2450 50  0001 C CNN
 F 4 "V" H 6400 2450 50  0001 C CNN "Spice_Primitive"
-F 5 "dc 15" H 6400 2450 50  0001 C CNN "Spice_Model"
+F 5 "dc 10" H 6400 2450 50  0001 C CNN "Spice_Model"
 F 6 "Y" H 6400 2450 50  0001 C CNN "Spice_Netlist_Enabled"
 	1    6400 2450
@@
 F 3 "~" H 6400 1650 50  0001 C CNN
 F 4 "V" H 6400 1650 50  0001 C CNN "Spice_Primitive"
-F 5 "dc 15" H 6400 1650 50  0001 C CNN "Spice_Model"
+F 5 "dc 10" H 6400 1650 50  0001 C CNN "Spice_Model"
 F 6 "Y" H 6400 1650 50  0001 C CNN "Spice_Netlist_Enabled"
 	1    6400 1650
@@
 F 2 "" H 4150 2050 50  0001 C CNN
 F 3 "~" H 4150 2050 50  0001 C CNN
-F 4 "R" H 4150 2050 50  0001 C CNN "Spice_Primitive"
-F 5 "0" H 4150 2050 50  0001 C CNN "Spice_Model"
+F 4 "X" H 4150 2050 50  0001 C CNN "Spice_Primitive"
+F 5 "TL082" H 4150 2050 50  0001 C CNN "Spice_Model"
 F 6 "Y" H 4150 2050 50  0001 C CNN "Spice_Netlist_Enabled"
-F 7 "adtl082_for_the_win.lib" H 4150 2050 50  0001 C CNN "Spice_Lib_File"
+F 7 "TL082.lib" H 4150 2050 50  0001 C CNN "Spice_Lib_File"
+F 8 "1 2 4 5 3" H 4150 2050 50  0001 C CNN "Spice_Node_Sequence"
 	1    4150 2050
 	1    0    0    -1
 $EndComp
+Wire Wire Line
+	3500 1950 3500 3000
+Wire Wire Line
+	2300 1500 2500 1500
+Wire Wire Line
+	2000 1500 1600 1500
+$Comp
+L Device:C C1
+U 1 1 6063BF78
+P 2150 1500
+F 0 "C1" V 1898 1500 50  0000 C CNN
+F 1 "470n" V 1989 1500 50  0000 C CNN
+F 2 "" H 2188 1350 50  0001 C CNN
+F 3 "~" H 2150 1500 50  0001 C CNN
+F 4 "C" H 2150 1500 50  0001 C CNN "Spice_Primitive"
+F 5 "470n" H 2150 1500 50  0001 C CNN "Spice_Model"
+F 6 "Y" H 2150 1500 50  0001 C CNN "Spice_Netlist_Enabled"
+	1    2150 1500
+	0    1    1    0
+$EndComp
 $EndSCHEMATC
